Commit message: Update jackal.urdf.xacro

File: src/jackal_description/urdf/jackal.urdf.xacro (robot description, xacro)
@@ -86,4 +86,10 @@
     <child link="chassis_link" />
   </joint>
+  <joint name="base_footprint_joint" type="fixed">
+    <origin xyz="0 0 0" rpy="0 0 0" />
+    <parent link="base_link"/>
+    <child link="base_footprint" />
+  </joint>
+  <link name="base_footprint"></link>
   <link name="chassis_link">
     <visual>
